File: min-eVOLVER/min-eV-PCB/min-evolver.kicad_sch (KiCad schematic)
At the start: 72 parts, among them CON1 BARREL_JACK, P1 CONN_02X12, P2 CONN_02X08, P3 CONN_02X08, P4 CONN_02X08, P7 CONN_01X02, Q1 Q_NMOS_GSD, Q10 Q_NMOS_GSD, Q11 Q_NMOS_GSD, Q12 Q_NMOS_GSD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

Commit message: min-eV PCBv1.2.2 better diode and mosfet footprints, corrected PCBway BOM (OD90 and OD135 resistors were swapped)
Parts:
- D1, D10, D11, D12, D2, D3, D4, D5, D6, D7, D8, D9: footprint mods:SBR160S23 -> min-eV-footprint-lib:diode_SBR160S23
- Q1, Q10, Q11, Q12, Q2, Q3, Q4, Q5, Q6, Q7, Q8, Q9: footprint mods:A03422 -> min-eV-footprint-lib:mosfet_A03422
